File: POWAH!.kicad_sch (KiCad schematic)
At the start: 22 parts, among them J5 PWR SUPPLY, U6 TSR1-2450E

Commit message: Last Push pour que tu check, après je commence le Layout
Parts:
- R15, R16, R17: value ? -> 10k
Changed lines of the file:
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@@
 			)
 		)
-		(property "Value" "?"
+		(property "Value" "10k"
 			(at 209.55 107.95 90)
 			(effects
@@
 			)
 		)
-		(property "Value" "?"
+		(property "Value" "10k"
 			(at 209.55 123.19 90)
 			(effects
@@
 			)
 		)
-		(property "Value" "?"
+		(property "Value" "10k"
 			(at 209.55 138.43 90)
 			(effects

Commit message: Finito je te laisse check
Parts:
- removed C33, C34, C35: ?, Capacitor_SMD:C_0402_1005Metric, symbol Device:C
- added J18: 24V_OUT_TO_BEC, Connector_JST:JST_VH_B2P-VH_1x02_P3.96mm_Vertical, symbol Connector:Conn_01x02_Pin
- added J19: BEC_8V4_IN, Connector_JST:JST_VH_B2P-VH_1x02_P3.96mm_Vertical, symbol Connector:Conn_01x02_Pin
- added R29: 0, Resistor_SMD:R_0805_2012Metric, symbol DPR_devices:R
- added R32, R33: 100k, Resistor_SMD:R_0603_1608Metric, symbol DPR_devices:R
Connections:
- net +24V: now also J18.1 (Pin_1)
- net GNDD: now also R29.2, R32.2, R33.2
- new net +8V4_SERVO: J19.1 (Pin_1)
- new net GND_SERVO: J18.2 (Pin_2), J19.2 (Pin_2), R29.1
- new net PWM_SERVO1: R32.1
- new net PWM_SERVO2: R33.1
Other:
- moved on the sheet: C27, C28, C32

Commit message: Changed M12 for SMA + 2 pins alim. --> we will have to split the cable from Kistlers
Changed lines of the file:
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@@
 	)
 	(junction
-		(at 238.76 64.77)
+		(at 43.18 60.96)
 		(diameter 0)
 		(color 0 0 0 0)
 	)
 	(junction
-		(at 227.33 64.77)
+		(at 238.76 64.77)
 		(diameter 0)
 		(color 0 0 0 0)
 	)
 	(junction
-		(at 238.76 74.93)
+		(at 227.33 64.77)
 		(diameter 0)
 		(color 0 0 0 0)
 	)
 	(junction
-		(at 43.18 60.96)
+		(at 238.76 74.93)
 		(diameter 0)
 		(color 0 0 0 0)
@@
 	(wire
 		(pts
-			(xy 41.91 60.96) (xy 43.18 60.96)
+			(xy 162.56 64.77) (xy 173.99 64.77)
 		)
 		(stroke
@@
 	(wire
 		(pts
-			(xy 162.56 64.77) (xy 173.99 64.77)
+			(xy 36.83 60.96) (xy 43.18 60.96)
 		)
 		(stroke
@@
 	(wire
 		(pts
+			(xy 43.18 60.96) (xy 43.18 64.77)
+		)
+		(stroke
+			(width 0)
+			(type default)
+		)
+	)
+	(wire
+		(pts
 			(xy 191.77 64.77) (xy 185.42 64.77)
 		)
@@
 	(wire
 		(pts
-			(xy 43.18 60.96) (xy 43.18 64.77)
-		)
-		(stroke
-			(width 0)
-			(type default)
-		)
-	)
-	(wire
-		(pts
 			(xy 43.18 67.31) (xy 43.18 76.2)
 		)
@@
 	)
 	(symbol
+		(lib_id "power:PWR_FLAG")
+		(at 36.83 60.96 90)
+		(unit 1)
+		(exclude_from_sim no)
+		(in_bom yes)
+		(on_board yes)
+		(dnp no)
+		(fields_autoplaced yes)
+		(property "Reference" "#FLG01"
+			(at 34.925 60.96 0)
+			(effects
+				(font
+					(size 1.27 1.27)
+				)
+				(hide yes)
+			)
+		)
+		(property "Value" "PWR_FLAG"
+			(at 33.02 60.9599 90)
+			(effects
+				(font
+					(size 1.27 1.27)
+				)
+				(justify left)
+			)
+		)
+		(property "Footprint" ""
+			(at 36.83 60.96 0)
+			(effects
+				(font
+					(size 1.27 1.27)
+				)
+				(hide yes)
+			)
+		)
+		(property "Datasheet" "~"
+			(at 36.83 60.96 0)
+			(effects
+				(font
+					(size 1.27 1.27)
+				)
+				(hide yes)
+			)
+		)
+		(property "Description" "Special symbol for telling ERC where power comes from"
+			(at 36.83 60.96 0)
+			(effects
+				(font
+					(size 1.27 1.27)
+				)
+				(hide yes)
+			)
+		)
+		(pin "1"
+		)
+		(instances
+			(project "Valvotron8000Pro"
+				(path "/e783bbdf-2a7f-40b9-9fb7-b62785862857/ce1b4cf9-39a0-46dc-88bb-a33de60f5f4c"
+					(reference "#FLG01")
+					(unit 1)
+				)
+			)
+		)
+	)
+	(symbol
 		(lib_id "power:+3V3")
 		(at 180.34 138.43 0)
@@
 					(unit 1)
 				)
-			)
-		)
-	)
-	(symbol
-		(lib_id "power:PWR_FLAG")
-		(at 41.91 60.96 90)
-		(unit 1)
-		(exclude_from_sim no)
-		(in_bom yes)
-		(on_board yes)
-		(dnp no)
-		(fields_autoplaced yes)
-		(property "Reference" "#FLG01"
-			(at 40.005 60.96 0)
-			(effects
-				(font
-					(size 1.27 1.27)
-				)
-				(hide yes)
-			)
-		)
-		(property "Value" "PWR_FLAG"
-			(at 38.1 60.9599 90)
-			(effects
-				(font
-					(size 1.27 1.27)
-				)
-				(justify left)
-			)
-		)
-		(property "Footprint" ""
-			(at 41.91 60.96 0)
-			(effects
-				(font
-					(size 1.27 1.27)
-				)
-				(hide yes)
-			)
-		)
-		(property "Datasheet" "~"
-			(at 41.91 60.96 0)
-			(effects
-				(font
-					(size 1.27 1.27)
-				)
-				(hide yes)
-			)
-		)
-		(property "Description" "Special symbol for telling ERC where power comes from"
-			(at 41.91 60.96 0)
-			(effects
-				(font
-					(size 1.27 1.27)
-				)
-				(hide yes)
-			)
-		)
-		(pin "1"
-		)
-		(instances
-			(project ""
-				(path "/e783bbdf-2a7f-40b9-9fb7-b62785862857/ce1b4cf9-39a0-46dc-88bb-a33de60f5f4c"
-					(reference "#FLG01")
-					(unit 1)
-				)

Commit message: Dernières modifs
Parts:
- J18, J19: footprint Connector_JST:JST_VH_B2P-VH_1x02_P3.96mm_Vertical -> Connector_JST:JST_XH_B2B-XH-AM_1x02_P2.50mm_Vertical
Changed lines of the file:
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@@
 			)
 		)
-		(property "Footprint" "Connector_JST:JST_VH_B2P-VH_1x02_P3.96mm_Vertical"
+		(property "Footprint" "Connector_JST:JST_XH_B2B-XH-AM_1x02_P2.50mm_Vertical"
 			(at 86.36 64.77 0)
 			(effects
@@
 			)
 		)
-		(property "Footprint" "Connector_JST:JST_VH_B2P-VH_1x02_P3.96mm_Vertical"
+		(property "Footprint" "Connector_JST:JST_XH_B2B-XH-AM_1x02_P2.50mm_Vertical"
 			(at 86.36 91.44 0)
 			(effects

Commit message: Changement des connecteurs servo (ne tenaient pas le courant en pics (=5A)) ++
Parts:
- J18, J19: footprint Connector_JST:JST_XH_B2B-XH-AM_1x02_P2.50mm_Vertical -> Connector_AMASS:AMASS_XT30U-F_1x02_P5.0mm_Vertical
Changed lines of the file:
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@@
 			)
 		)
-		(property "Footprint" "Connector_JST:JST_XH_B2B-XH-AM_1x02_P2.50mm_Vertical"
+		(property "Footprint" "Connector_AMASS:AMASS_XT30U-F_1x02_P5.0mm_Vertical"
 			(at 86.36 64.77 0)
 			(effects
@@
 			)
 		)
-		(property "Footprint" "Connector_JST:JST_XH_B2B-XH-AM_1x02_P2.50mm_Vertical"
+		(property "Footprint" "Connector_AMASS:AMASS_XT30U-F_1x02_P5.0mm_Vertical"
 			(at 86.36 91.44 0)
 			(effects
