File: CAN_interface.kicad_sch (KiCad schematic)
At the start: 24 parts, among them J3 CAN_OUT, J4 CAN_IN, U4 MCP2515-xST, U5 MCP2551-I-SN, Y3 Crystal_GND24

Commit message: Last Push pour que tu check, après je commence le Layout
Other:
- note added: "Connectors"
Changed lines of the file:
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@@
 	(generator_version "9.0")
 	(paper "A4")
+	(text "Connectors\n"
+		(exclude_from_sim no)
+		(at 221.742 62.738 0)
+		(effects
+			(font
+				(size 1.27 1.27)
+			)
+		)
+	)
 	(junction
 		(at 143.51 161.29)
@@
 			)
 			(justify left bottom)
-		)
-	)
-	(label "Connectors"
-		(at 213.36 63.5 0)
-		(effects
-			(font
-				(size 1.27 1.27)
-				(color 255 0 255 1)
-			)
-			(justify left bottom)

Commit message: Finito je te laisse check
Other:
- note added: "50~100R 100MHz"
- note added: "A FAIRE : CONNECTEUR CAN CONNECTEUR M12 + SMA"
- note added: "Crystal close to chip pls"
- note added: "RC for auto reset"
- note added: "Signal protection and conditioning"
- note added: "Some bypass around here, IDK man I'm just vide KiCading at this point"
- note added: "TVS diode array"
- note added: "only for termination"
- note added: "remove jumper after debugging"
- note added: "should be VDD/2"
Changed lines of the file:
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@@
 	(generator_version "9.0")
 	(paper "A4")
+	(text "TVS diode array\n"
+		(exclude_from_sim no)
+		(at 116.078 173.482 0)
+		(effects
+			(font
+				(size 1.27 1.27)
+			)
+		)
+	)
+	(text "50~100R 100MHz"
+		(exclude_from_sim no)
+		(at 110.744 169.672 0)
+		(effects
+			(font
+				(size 1.27 1.27)
+			)
+		)
+	)
 	(text "Connectors\n"
 		(exclude_from_sim no)
@@
 		)
 	)
+	(text "Some bypass around here, IDK man I'm just vide KiCading at this point"
+		(exclude_from_sim no)
+		(at 132.08 25.908 0)
+		(effects
+			(font
+				(size 1.27 1.27)
+			)
+		)
+	)
+	(text "should be VDD/2"
+		(exclude_from_sim no)
+		(at 31.496 154.94 0)
+		(effects
+			(font
+				(size 1.27 1.27)
+			)
+		)
+	)
+	(text "Signal protection and conditioning"
+		(exclude_from_sim no)
+		(at 108.966 153.416 0)
+		(effects
+			(font
+				(size 1.27 1.27)
+			)
+		)
+	)
+	(text "A FAIRE : CONNECTEUR CAN\nCONNECTEUR M12 + SMA\n"
+		(exclude_from_sim no)
+		(at 238.76 36.322 0)
+		(effects
+			(font
+				(size 1.27 1.27)
+			)
+		)
+	)
+	(text "RC for auto reset\n"
+		(exclude_from_sim no)
+		(at 152.4 57.658 0)
+		(effects
+			(font
+				(size 1.27 1.27)
+			)
+		)
+	)
+	(text "remove jumper after debugging"
+		(exclude_from_sim no)
+		(at 69.342 36.83 0)
+		(effects
+			(font
+				(size 1.27 1.27)
+			)
+		)
+	)
+	(text "Crystal close to chip pls"
+		(exclude_from_sim no)
+		(at 57.658 75.438 0)
+		(effects
+			(font
+				(size 1.27 1.27)
+			)
+		)
+	)
+	(text "only for termination\n\n\n"
+		(exclude_from_sim no)
+		(at 144.78 160.782 0)
+		(effects
+			(font
+				(size 1.27 1.27)
+			)
+		)
+	)
 	(junction
 		(at 143.51 161.29)
@@
 	(junction
 		(at 124.46 33.02)
+		(diameter 0)
+		(color 0 0 0 0)
+	)
+	(junction
+		(at 91.44 100.33)
 		(diameter 0)
 		(color 0 0 0 0)
@@
 	(wire
 		(pts
+			(xy 91.44 100.33) (xy 91.44 97.79)
+		)
+		(stroke
+			(width 0)
+			(type default)
+		)
+	)
+	(wire
+		(pts
 			(xy 151.13 167.64) (xy 151.13 168.91)
 		)
@@
 	(wire
 		(pts
+			(xy 88.9 100.33) (xy 91.44 100.33)
+		)
+		(stroke
+			(width 0)
+			(type default)
+		)
+	)
+	(wire
+		(pts
 			(xy 91.44 33.02) (xy 91.44 57.15)
 		)
@@
 	(wire
 		(pts
-			(xy 91.44 104.14) (xy 91.44 97.79)
+			(xy 91.44 104.14) (xy 91.44 100.33)
 		)
 		(stroke
@@
 			(width 0)
 			(type default)
-		)
-	)
-	(label "should be VDD{slash}2"
-		(at 27.94 156.21 0)
-		(effects
-			(font
-				(size 1.27 1.27)
-			)
-			(justify left bottom)
-		)
-	)
-	(label "Some bypass around here, IDK man I'm just vide KiCading at this point"
-		(at 95.25 26.67 0)
-		(effects
-			(font
-				(size 1.27 1.27)
-				(color 0 0 194 1)
-			)
-			(justify left bottom)
 		)
 	)
@@
 		)
 	)
-	(label "Signal protection and conditioning"
-		(at 90.17 153.67 0)
-		(effects
-			(font
-				(size 1.27 1.27)
-				(color 255 0 0 1)
-			)
-			(justify left bottom)
-		)
-	)
-	(label "TVS diode array"
-		(at 97.79 172.72 0)
-		(effects
-			(font
-				(size 1.27 1.27)
-			)
-			(justify left bottom)
-		)
-	)
-	(label "remove jumper after debugging"
-		(at 57.15 38.1 0)
-		(effects
-			(font
-				(size 1.27 1.27)
-			)
-			(justify left bottom)
-		)
-	)
-	(label "RC for auto reset"
-		(at 143.51 58.42 0)
-		(effects
-			(font
-				(size 1.27 1.27)
-				(color 0 194 0 1)
-			)
-			(justify left bottom)
-		)
-	)
 	(label "Shield"
 		(at 243.84 92.71 0)
-		(effects
-			(font
-				(size 1.27 1.27)
-			)
-			(justify left bottom)
-		)
-	)
-	(label "only for termination"
-		(at 134.62 160.02 0)
-		(effects
-			(font
-				(size 1.27 1.27)
-			)
-			(justify left bottom)
-		)
-	)
-	(label "50~100R 100MHz"
-		(at 102.87 170.18 0)
-		(effects
-			(font
-				(size 1.27 1.27)
-			)
-			(justify left bottom)
-		)
-	)
-	(label "Crystal close to chip pls"
-		(at 45.72 76.2 0)
 		(effects
 			(font
@@
 			(fill
 				(type none)
+			)
+		)
+	)
+	(rule_area
+		(polyline
+			(pts
+				(xy 223.52 31.75) (xy 255.27 31.75) (xy 255.27 40.64) (xy 226.06 40.64) (xy 223.52 38.1)
+			)
+			(stroke
+				(width 1)
+				(type solid)
+				(color 194 0 0 1)
+			)
+			(fill
+				(type color)
+				(color 255 0 0 0.29)
 			)
 		)
@@
 					(unit 1)
 				)
+			)
+		)
+	)
+	(symbol
+		(lib_id "power:PWR_FLAG")
+		(at 88.9 100.33 90)
+		(unit 1)
+		(exclude_from_sim no)
+		(in_bom yes)
+		(on_board yes)
+		(dnp no)
+		(fields_autoplaced yes)
+		(property "Reference" "#FLG02"
+			(at 86.995 100.33 0)
+			(effects
+				(font
+					(size 1.27 1.27)
+				)
+				(hide yes)
+			)
+		)
+		(property "Value" "PWR_FLAG"
+			(at 85.09 100.3299 90)
+			(effects
+				(font
+					(size 1.27 1.27)
+				)
+				(justify left)
+			)
+		)
+		(property "Footprint" ""
+			(at 88.9 100.33 0)
+			(effects
+				(font
+					(size 1.27 1.27)
+				)
+				(hide yes)
+			)
+		)
+		(property "Datasheet" "~"
+			(at 88.9 100.33 0)
+			(effects
+				(font
+					(size 1.27 1.27)
+				)
+				(hide yes)
+			)
+		)
+		(property "Description" "Special symbol for telling ERC where power comes from"
+			(at 88.9 100.33 0)
+			(effects
+				(font
+					(size 1.27 1.27)
+				)
+				(hide yes)
+			)
+		)
+		(pin "1"
+		)
+		(instances
+			(project ""
+				(path "/e783bbdf-2a7f-40b9-9fb7-b62785862857/ab3725e4-8594-4005-8898-2e8169b9e1ee"
+					(reference "#FLG02")
+					(unit 1)
+				)

Commit message: last modifications
Other:
- note removed: "A FAIRE : CONNECTEUR CAN CONNECTEUR M12 + SMA"
Changed lines of the file:
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@@
-		)
-	)
-	(text "A FAIRE : CONNECTEUR CAN\nCONNECTEUR M12 + SMA\n"
-		(exclude_from_sim no)
-		(at 238.76 36.322 0)
-		(effects
-			(font
-				(size 1.27 1.27)
-			)
 		)
 	)
@@
 			)
 		)
-	)
-	(rule_area
-		(polyline
-			(pts
-				(xy 223.52 31.75) (xy 255.27 31.75) (xy 255.27 40.64) (xy 226.06 40.64) (xy 223.52 38.1)
-			)
-			(stroke
-				(width 1)
-				(type solid)
-				(color 194 0 0 1)
-			)
-			(fill
-				(type color)
-				(color 255 0 0 0.29)
-			)
-		)

Commit message: Changed M12 for SMA + 2 pins alim. --> we will have to split the cable from Kistlers
Changed lines of the file:
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@@
-	)
-	(junction
-		(at 91.44 100.33)
-		(diameter 0)
-		(color 0 0 0 0)
 	)
 	(junction
@@
 	(wire
 		(pts
+			(xy 91.44 97.79) (xy 91.44 104.14)
+		)
+		(stroke
+			(width 0)
+			(type default)
+		)
+	)
+	(wire
+		(pts
 			(xy 142.24 90.17) (xy 142.24 92.71)
 		)
@@
 	(wire
 		(pts
-			(xy 91.44 100.33) (xy 91.44 97.79)
-		)
-		(stroke
-			(width 0)
-			(type default)
-		)
-	)
-	(wire
-		(pts
 			(xy 151.13 167.64) (xy 151.13 168.91)
 		)
@@
 	(wire
 		(pts
-			(xy 88.9 100.33) (xy 91.44 100.33)
-		)
-		(stroke
-			(width 0)
-			(type default)
-		)
-	)
-	(wire
-		(pts
 			(xy 91.44 33.02) (xy 91.44 57.15)
 		)
@@
 		(pts
 			(xy 69.85 85.09) (xy 76.2 85.09)
-		)
-		(stroke
-			(width 0)
-			(type default)
-		)
-	)
-	(wire
-		(pts
-			(xy 91.44 104.14) (xy 91.44 100.33)
 		)
 		(stroke
@@
 					(unit 1)
 				)
-			)
-		)
-	)
-	(symbol
-		(lib_id "power:PWR_FLAG")
-		(at 88.9 100.33 90)
-		(unit 1)
-		(exclude_from_sim no)
-		(in_bom yes)
-		(on_board yes)
-		(dnp no)
-		(fields_autoplaced yes)
-		(property "Reference" "#FLG02"
-			(at 86.995 100.33 0)
-			(effects
-				(font
-					(size 1.27 1.27)
-				)
-				(hide yes)
-			)
-		)
-		(property "Value" "PWR_FLAG"
-			(at 85.09 100.3299 90)
-			(effects
-				(font
-					(size 1.27 1.27)
-				)
-				(justify left)
-			)
-		)
-		(property "Footprint" ""
-			(at 88.9 100.33 0)
-			(effects
-				(font
-					(size 1.27 1.27)
-				)
-				(hide yes)
-			)
-		)
-		(property "Datasheet" "~"
-			(at 88.9 100.33 0)
-			(effects
-				(font
-					(size 1.27 1.27)
-				)
-				(hide yes)
-			)
-		)
-		(property "Description" "Special symbol for telling ERC where power comes from"
-			(at 88.9 100.33 0)
-			(effects
-				(font
-					(size 1.27 1.27)
-				)
-				(hide yes)
-			)
-		)
-		(pin "1"
-		)
-		(instances
-			(project ""
-				(path "/e783bbdf-2a7f-40b9-9fb7-b62785862857/ab3725e4-8594-4005-8898-2e8169b9e1ee"
-					(reference "#FLG02")
-					(unit 1)
-				)

Commit message: changed the mcp - potentiellement final version
Parts:
- removed C17, C24: 10n, Capacitor_SMD:C_0402_1005Metric, symbol Device:C
- removed C18: 10u, Capacitor_SMD:C_0805_2012Metric, symbol Device:C
- removed C19: 1u, Capacitor_SMD:C_0603_1608Metric, symbol Device:C
- removed C3: 100n, Capacitor_SMD:C_0402_1005Metric, symbol Device:C
- removed D2: VCAN36A2-03G-E3-08, KiNic_footprints:SOT65P230X110-3N, symbol KiNic_symbols:VCAN36A2-03G-E3-08
- removed FL1: Common mode choke, KiNic_footprints:DLW21SN121HQ2L, symbol Device:Filter_EMI_CommonMode
- removed R7, R8: 10k, Resistor_SMD:R_0603_1608Metric, symbol Device:R_US
- removed R9: 120, Resistor_SMD:R_0603_1608Metric, symbol Device:R_US
- removed TP4: Vref, TestPoint:TestPoint_Pad_D2.0mm, symbol Connector:TestPoint
- removed U4: MCP2515-xST, Package_SO:TSSOP-20_4.4x6.5mm_P0.65mm, symbol Interface_CAN_LIN:MCP2515-xST
- removed U5: MCP2551-I-SN, Package_SO:SOIC-8_3.9x4.9mm_P1.27mm, symbol Interface_CAN_LIN:MCP2551-I-SN
- added D?: VCAN36A2-03G-E3-08, KiNic_footprints:SOT65P230X110-3N, symbol KiNic_symbols:VCAN36A2-03G-E3-08
- added FL?: Common mode choke, KiNic_footprints:DLW21SN121HQ2L, symbol Device:Filter_EMI_CommonMode
- added R?: 120, Resistor_SMD:R_0603_1608Metric, symbol Device:R_US
- added R? (x2): 10k, Resistor_SMD:R_0603_1608Metric, symbol Device:R_US
- added U?: MCP25625x-x-ML, Package_DFN_QFN:QFN-28-1EP_6x6mm_P0.65mm_EP4.25x4.25mm, symbol Interface_CAN_LIN:MCP25625x-x-ML
Connections:
- net +3V3: now also R?.1, R?.1
- net +5V: now also U?.19 (V_{DDA})
- net CANH: now also FL?.2, R?.1
- net CANL: now also FL?.4, R?.2
- net GNDD: now also D?.3, U?.18 (V_{SS}), U?.22 (GND)
- net INT: now also R?.2, U?.25 (~{INT})
- net MISO: now also U?.28 (SO)
- net MOSI: now also U?.27 (SI)
- net RESET_CAN: now also U?.2 (~{RESET})
- net SCLK: now also U?.26 (SCK)
- net SS: now also R?.2, U?.1 (~{CS})
- net at C20.1, Y3.2: now also U?.20 (OSC2)
- net at C21.1, Y3.4: now also U?.21 (OSC1)
- new net: D?.1, FL?.1, U?.13 (CANH)
- new net: D?.2, FL?.3, U?.12 (CANL)
- new net: U?.10 (R_{XD}), U?.5 (RxCAN)
- new net: U?.16 (T_{XD}), U?.4 (TxCAN)
- new net +3.3V: U?.11 (V_{IO}), U?.3 (V_{DD})
- new net GND: U?.15 (STBY)
- no-connect marks 7 -> 8
Other:
- note added: "C23 (100nF) must be very close to pin 19 !"
- note added: "New CAN disposition (all in one bro) Compatible with RP2040 - Thanks to DPR"
- note removed: "RC for auto reset"
- note removed: "Some bypass around here, IDK man I'm just vide KiCading at this point"
- note removed: "remove jumper after debugging"
- note removed: "should be VDD/2"
- moved on the sheet: C20, C21, C22, C23, C25, C26, D1, J3, J4, R6, Y3

Commit message: Layout done, pcb ready (finally)
Parts:
- gave numbers to parts that had none: 6
Connections:
- net GNDD: now also U4.29 (EP)
