File: DPR_devices.kicad_sch (KiCad schematic)
At the start: 54 parts, among them J10 SMA_K2, J11 SMA_K3, J12 Sens. P2, J13 Sens. P3, J14 Servo1, J16 Servo2, J17 Sens. P1, J6 PWR_K1, J7 PWR_K2, J8 PWR_K3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

Commit message: Dernières modifs
Parts:
- removed R23, R24, R25, R26, R27, R28: 4.7k, Resistor_SMD:R_0603_1608Metric, symbol DPR_devices:R
- added H1, H2, H4: MountingHole, MountingHole:MountingHole_2.5mm, symbol Mechanical:MountingHole
- added R23, R24, R25, R26, R27, R28: 4.7k, Resistor_SMD:R_0603_1608Metric, symbol Device:R
- J6, J7, J8: footprint Connector_JST:JST_GH_BM02B-GHS-TBT_1x02-1MP_P1.25mm_Vertical -> Connector_JST:JST_XH_B2B-XH-AM_1x02_P2.50mm_Vertical
Connections:
- net +3V3: now also R23.2, R24.1, R25.2, R26.1, R27.2, R28.1; no longer J12.1, J12.2, J13.1, J13.2, J17.1, J17.2
- net PTE1_SCL: now also J17.1, R27.1
- net PTE1_SDA: now also J17.2, R28.2
- net PTE2_SCL: now also J12.1, R23.1
- net PTE2_SDA: now also J12.2, R24.2
- net PTE3_SCL: now also J13.1, R25.1
- net PTE3_SDA: now also J13.2, R26.2

Commit message: Changement des connecteurs servo (ne tenaient pas le courant en pics (=5A)) ++
Parts:
- J14, J16: footprint Connector_PinHeader_2.54mm:PinHeader_1x03_P2.54mm_Vertical -> Connector_Phoenix_MSTB:PhoenixContact_MSTBVA_2,5_3-G_1x03_P5.00mm_Vertical
Changed lines of the file:
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@@
 			)
 		)
-		(property "Footprint" "Connector_PinHeader_2.54mm:PinHeader_1x03_P2.54mm_Vertical"
+		(property "Footprint" "Connector_Phoenix_MSTB:PhoenixContact_MSTBVA_2,5_3-G_1x03_P5.00mm_Vertical"
 			(at 161.29 139.7 0)
 			(effects
@@
 			)
 		)
-		(property "Footprint" "Connector_PinHeader_2.54mm:PinHeader_1x03_P2.54mm_Vertical"
+		(property "Footprint" "Connector_Phoenix_MSTB:PhoenixContact_MSTBVA_2,5_3-G_1x03_P5.00mm_Vertical"
 			(at 161.29 154.94 0)
 			(effects

Commit message: Layout done, pcb ready (finally)
Other:
- moved on the sheet: H1, H2, H4
Changed lines of the file:
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@@
 		(polyline
 			(pts
-				(xy 262.89 156.21) (xy 211.455 156.21) (xy 209.55 153.67) (xy 209.55 130.81) (xy 262.89 130.81)
+				(xy 250.19 156.21) (xy 199.39 156.21) (xy 199.39 153.67) (xy 199.39 130.81) (xy 250.19 130.81)
 			)
 			(stroke
@@
 		(polyline
 			(pts
-				(xy 16.51 25.4) (xy 16.51 130.81) (xy 20.32 134.62) (xy 101.6 134.62) (xy 109.22 127) (xy 109.22 82.55)
-				(xy 113.03 78.74) (xy 194.31 78.74) (xy 203.2 69.85) (xy 203.2 19.05) (xy 22.86 19.05)
+				(xy 16.51 25.4) (xy 16.51 130.81) (xy 20.32 134.62) (xy 101.6 134.62) (xy 109.22 127) (xy 109.22 86.36)
+				(xy 114.3 81.28) (xy 205.74 81.28) (xy 205.74 73.66) (xy 205.74 20.32) (xy 22.86 19.05)
 			)
 			(stroke
@@
 	(symbol
 		(lib_id "Mechanical:MountingHole")
-		(at 215.9 149.86 0)
+		(at 205.74 149.86 0)
 		(unit 1)
 		(exclude_from_sim no)
@@
 		(fields_autoplaced yes)
 		(property "Reference" "H2"
-			(at 218.44 148.5899 0)
+			(at 208.28 148.5899 0)
 			(effects
 				(font
@@
 		)
 		(property "Value" "MountingHole"
-			(at 218.44 151.1299 0)
+			(at 208.28 151.1299 0)
 			(effects
 				(font
@@
 		)
 		(property "Footprint" "MountingHole:MountingHole_2.5mm"
-			(at 215.9 149.86 0)
+			(at 205.74 149.86 0)
 			(effects
 				(font
@@
 		)
 		(property "Datasheet" "~"
-			(at 215.9 149.86 0)
+			(at 205.74 149.86 0)
 			(effects
 				(font
@@
 		)
 		(property "Description" "Mounting Hole without connection"
-			(at 215.9 149.86 0)
+			(at 205.74 149.86 0)
 			(effects
 				(font
@@
 	(symbol
 		(lib_id "Mechanical:MountingHole")
-		(at 241.3 149.86 0)
+		(at 231.14 149.86 0)
 		(unit 1)
 		(exclude_from_sim no)
@@
 		(fields_autoplaced yes)
 		(property "Reference" "H4"
-			(at 243.84 148.5899 0)
+			(at 233.68 148.5899 0)
 			(effects
 				(font
@@
 		)
 		(property "Value" "MountingHole"
-			(at 243.84 151.1299 0)
+			(at 233.68 151.1299 0)
 			(effects
 				(font
@@
 		)
 		(property "Footprint" "MountingHole:MountingHole_2.5mm"
-			(at 241.3 149.86 0)
+			(at 231.14 149.86 0)
 			(effects
 				(font
@@
 		)
 		(property "Datasheet" "~"
-			(at 241.3 149.86 0)
+			(at 231.14 149.86 0)
 			(effects
 				(font
@@
 		)
 		(property "Description" "Mounting Hole without connection"
-			(at 241.3 149.86 0)
+			(at 231.14 149.86 0)
 			(effects
 				(font
@@
 	(symbol
 		(lib_id "Mechanical:MountingHole")
-		(at 215.9 137.16 0)
+		(at 205.74 137.16 0)
 		(unit 1)
 		(exclude_from_sim no)
@@
 		(fields_autoplaced yes)
 		(property "Reference" "H1"
-			(at 218.44 135.8899 0)
+			(at 208.28 135.8899 0)
 			(effects
 				(font
@@
 		)
 		(property "Value" "MountingHole"
-			(at 218.44 138.4299 0)
+			(at 208.28 138.4299 0)
 			(effects
 				(font
@@
 		)
 		(property "Footprint" "MountingHole:MountingHole_2.5mm"
-			(at 215.9 137.16 0)
+			(at 205.74 137.16 0)
 			(effects
 				(font
@@
 		)
 		(property "Datasheet" "~"
-			(at 215.9 137.16 0)
+			(at 205.74 137.16 0)
 			(effects
 				(font
@@
 		)
 		(property "Description" "Mounting Hole without connection"
-			(at 215.9 137.16 0)
+			(at 205.74 137.16 0)
 			(effects
 				(font
